File: Battery_Storage_Device.sch (KiCad schematic (older format))
At the start: 47 parts, among them J4 Barrel_Jack_Switch, K1 EE2-5NU, Q1 MMBT5551L, Q2 MMBT5551L, Q3 Q_PMOS_GDS, Q4 Q_PMOS_GDS, Q5 BSS138, U1 TLV2372, U11 LM317_SOT-223, U2 TLV2372

Commit message: New power banana jacks, general updates
Parts:
- added D18, D19: 10V, Diode_SMD:D_SOD-123, symbol Device:D_Zener
- added TP1, TP2, TP3, TP4, TP5: TestPoint, TestPoint:TestPoint_THTPad_D2.0mm_Drill1.0mm, symbol Connector:TestPoint
- C1, C2: value 10n -> 0.1u
- D14: symbol Diode:MBRA340 -> Battery_Storage_Device-rescue:MBRA340-Diode
- H1, H2, H3, H4: footprint MountingHole:MountingHole_3.7mm_Pad -> MountingHole:MountingHole_2.7mm_M2.5_Pad
- K1: symbol Relay:EE2-5NU -> Battery_Storage_Device-rescue:EE2-5NU-Relay
- R17, R18: value 1M -> 100k
- R3, R4: value 100k -> 1M
- U11: symbol Regulator_Linear:LM317_SOT-223 -> Battery_Storage_Device-rescue:LM317_SOT-223-Regulator_Linear
Connections:
- net SRC_SINK: now also D19.1 (K), TP3.1
- net at Q4.1 (G), R12.2, R17.2: now also D19.2 (A)
- net at R7.2, U2.2 (-), U2.7: now also TP5.1
- net at C4.1, R4.2, U2.3 (+): now also TP4.1
- net at R8.1, U1.2 (-), U1.7: now also TP1.1
- net at C3.1, R3.2, U1.3 (+): now also TP2.1
- net at Q3.1 (G), R14.2, R18.2: now also D18.2 (A)
- net at Q3.3 (S), R16.2, R18.1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: now also D18.1 (K)
Other:
- moved on the sheet: C6, Q1, Q2, R12, R14, R17, R5, R6
