File: battery_afe.sch (KiCad schematic (older format))
At the start: 65 parts, among them J1 Conn_01x02_Female, J2 Conn_01x07_Male, Q10 BSS84, Q11 BSS84, Q12 BSS138, Q13 BSS138, Q14 BSS84, Q15 BSS138, Q16 BSS84, Q17 BSS138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

Commit message: Updates to the AFE power scheme to prevent discharging of the batteries
Parts:
- added C28: 10n, Capacitor_SMD:C_0805_2012Metric, symbol Device:C
- added R47: 10M, Resistor_SMD:R_0805_2012Metric, symbol Device:R_US
- added R48: 2M, Resistor_SMD:R_0805_2012Metric, symbol Device:R_US
Connections:
- net +BATT: now also R47.2; no longer C16.1, C7.1, C8.1, U3.13 (V+), U4.13 (V+), U5.13 (V+)
- net GND: now also C28.2, R48.1
- net at U7.7 (AIN2): now also C28.1, R47.1, R48.2
- new net +24V: C16.1, C7.1, C8.1, U3.13 (V+), U4.13 (V+), U5.13 (V+)
Other:
- moved on the sheet: U5D
Changed lines of the file:
@@
-	1    0    0    -1
-$EndComp
-$Comp
-L power:+BATT #PWR026
-U 1 1 5F76DBC6
-P 2850 3100
-F 0 "#PWR026" H 2850 2950 50  0001 C CNN
-F 1 "+BATT" H 2865 3273 50  0000 C CNN
-F 2 "" H 2850 3100 50  0001 C CNN
-F 3 "" H 2850 3100 50  0001 C CNN
-	1    2850 3100
 	1    0    0    -1
 $EndComp
@@
 Wire Wire Line
 	2850 1100 2850 1200
-$Comp
-L power:+BATT #PWR025
-U 1 1 5F7437F4
-P 2850 1100
-F 0 "#PWR025" H 2850 950 50  0001 C CNN
-F 1 "+BATT" H 2865 1273 50  0000 C CNN
-F 2 "" H 2850 1100 50  0001 C CNN
-F 3 "" H 2850 1100 50  0001 C CNN
-	1    2850 1100
-	1    0    0    -1
-$EndComp
 $Comp
 L power:GND #PWR021
@@
 	10350 4850 10350 4600
 Connection ~ 10350 4850
-$Comp
-L power:+BATT #PWR043
-U 1 1 5F7FD35F
-P 10350 4600
-F 0 "#PWR043" H 10350 4450 50  0001 C CNN
-F 1 "+BATT" H 10365 4773 50  0000 C CNN
-F 2 "" H 10350 4600 50  0001 C CNN
-F 3 "" H 10350 4600 50  0001 C CNN
-	1    10350 4600
-	1    0    0    -1
-$EndComp
 Wire Wire Line
 	9950 4850 9900 4850
@@
 	7500 2100 7500 1850
 Wire Wire Line
-	7500 1850 7700 1850
-Wire Wire Line
-	7700 1850 7700 1900
+	7500 1850 7350 1850
+Wire Wire Line
+	7350 1850 7350 1900
 $Comp
 L power:GND #PWR036
 U 1 1 5FF0AC73
-P 7700 1900
-F 0 "#PWR036" H 7700 1650 50  0001 C CNN
-F 1 "GND" H 7705 1727 50  0000 C CNN
-F 2 "" H 7700 1900 50  0001 C CNN
-F 3 "" H 7700 1900 50  0001 C CNN
-	1    7700 1900
+P 7350 1900
+F 0 "#PWR036" H 7350 1650 50  0001 C CNN
+F 1 "GND" H 7355 1727 50  0000 C CNN
+F 2 "" H 7350 1900 50  0001 C CNN
+F 3 "" H 7350 1900 50  0001 C CNN
+	1    7350 1900
 	1    0    0    -1
 $EndComp
@@
 Wire Wire Line
 	1100 900  1450 900
-$Comp
-L Analog_Switch:DG412xY U5
-U 4 1 61A0257A
-P 7500 1000
-F 0 "U5" H 7500 1267 50  0000 C CNN
-F 1 "DG412xY" H 7500 1176 50  0000 C CNN
-F 2 "Package_SO:SOIC-16_3.9x9.9mm_P1.27mm" H 7500 900 50  0001 C CNN
-F 3 "https://datasheets.maximintegrated.com/en/ds/DG411-DG413.pdf" H 7500 1000 50  0001 C CNN
-	4    7500 1000
-	1    0    0    -1
-$EndComp
-$Comp
-L power:GND #PWR0102
-U 1 1 61A7285A
-P 7500 1200
-F 0 "#PWR0102" H 7500 950 50  0001 C CNN
-F 1 "GND" H 7505 1027 50  0000 C CNN
-F 2 "" H 7500 1200 50  0001 C CNN
-F 3 "" H 7500 1200 50  0001 C CNN
-	1    7500 1200
-	1    0    0    -1
-$EndComp
-NoConn ~ 7200 1000
-NoConn ~ 7800 1000
 Text HLabel 1450 900  2    50   BiDi ~ 0
 PACK_HI
@@
 Wire Wire Line
 	4100 2450 4200 2450
+$Comp
+L power:GND #PWR0102
+U 1 1 61A7285A
+P 7050 1250
+F 0 "#PWR0102" H 7050 1000 50  0001 C CNN
+F 1 "GND" H 7055 1077 50  0000 C CNN
+F 2 "" H 7050 1250 50  0001 C CNN
+F 3 "" H 7050 1250 50  0001 C CNN
+	1    7050 1250
+	1    0    0    -1
+$EndComp
+$Comp
+L Analog_Switch:DG412xY U5
+U 4 1 61A0257A
+P 7050 1050
+F 0 "U5" H 7050 1317 50  0000 C CNN
+F 1 "DG412xY" H 7050 1226 50  0000 C CNN
+F 2 "Package_SO:SOIC-16_3.9x9.9mm_P1.27mm" H 7050 950 50  0001 C CNN
+F 3 "https://datasheets.maximintegrated.com/en/ds/DG411-DG413.pdf" H 7050 1050 50  0001 C CNN
+	4    7050 1050
+	1    0    0    -1
+$EndComp
+NoConn ~ 6750 1050
+NoConn ~ 7350 1050
+$Comp
+L Device:R_US R?
+U 1 1 5F860D69
+P 7800 1600
+AR Path="/5F860D69" Ref="R?"  Part="1"
+AR Path="/5F71FE73/5F860D69" Ref="R48"  Part="1"
+F 0 "R48" H 7868 1646 50  0000 L CNN
+F 1 "2M" H 7868 1555 50  0000 L CNN
+F 2 "Resistor_SMD:R_0805_2012Metric" V 7840 1590 50  0001 C CNN
+F 3 "~" H 7800 1600 50  0001 C CNN
+	1    7800 1600
+	-1   0    0    1
+$EndComp
+$Comp
+L Device:R_US R?
+U 1 1 5F87874E
+P 7800 1150
+AR Path="/5F87874E" Ref="R?"  Part="1"
+AR Path="/5F71FE73/5F87874E" Ref="R47"  Part="1"
+F 0 "R47" H 7868 1196 50  0000 L CNN
+F 1 "10M" H 7868 1105 50  0000 L CNN
+F 2 "Resistor_SMD:R_0805_2012Metric" V 7840 1140 50  0001 C CNN
+F 3 "~" H 7800 1150 50  0001 C CNN
+	1    7800 1150
+	-1   0    0    1
+$EndComp
+$Comp
+L Device:C C28
+U 1 1 5F8C5990
+P 8150 1600
+F 0 "C28" V 7898 1600 50  0000 C CNN
+F 1 "10n" V 7989 1600 50  0000 C CNN
+F 2 "Capacitor_SMD:C_0805_2012Metric" H 8188 1450 50  0001 C CNN
+F 3 "~" H 8150 1600 50  0001 C CNN
+	1    8150 1600
+	1    0    0    -1
+$EndComp
+Wire Wire Line
+	8150 1450 8150 1350
+Wire Wire Line
+	8150 1350 7800 1350
+Wire Wire Line
+	7800 1350 7800 1300
+Wire Wire Line
+	7800 1450 7800 1350
+Connection ~ 7800 1350
+Wire Wire Line
+	7800 1000 7800 850
+$Comp
+L power:GND #PWR080
+U 1 1 5F94472F
+P 7800 1750
+F 0 "#PWR080" H 7800 1500 50  0001 C CNN
+F 1 "GND" H 7805 1577 50  0000 C CNN
+F 2 "" H 7800 1750 50  0001 C CNN
+F 3 "" H 7800 1750 50  0001 C CNN
+	1    7800 1750
+	1    0    0    -1
+$EndComp
+$Comp
+L power:GND #PWR081
+U 1 1 5F95C397
+P 8150 1750
+F 0 "#PWR081" H 8150 1500 50  0001 C CNN
+F 1 "GND" H 8155 1577 50  0000 C CNN
+F 2 "" H 8150 1750 50  0001 C CNN
+F 3 "" H 8150 1750 50  0001 C CNN
+	1    8150 1750
+	1    0    0    -1
+$EndComp
+Wire Wire Line
+	8150 1350 8400 1350
+Wire Wire Line
+	8400 1350 8400 2800
+Wire Wire Line
+	8400 2800 8750 2800
+Connection ~ 8150 1350
+$Comp
+L power:+24V #PWR?
+U 1 1 5FA77155
+P 2850 1100
+AR Path="/5FA77155" Ref="#PWR?"  Part="1"
+AR Path="/5F71FE73/5FA77155" Ref="#PWR0101"  Part="1"
+F 0 "#PWR0101" H 2850 950 50  0001 C CNN
+F 1 "+24V" H 2865 1273 50  0000 C CNN
+F 2 "" H 2850 1100 50  0001 C CNN
+F 3 "" H 2850 1100 50  0001 C CNN
+	1    2850 1100
+	1    0    0    -1
+$EndComp
+$Comp
+L power:+24V #PWR?
+U 1 1 5FA94618
+P 2850 3100
+AR Path="/5FA94618" Ref="#PWR?"  Part="1"
+AR Path="/5F71FE73/5FA94618" Ref="#PWR0107"  Part="1"
+F 0 "#PWR0107" H 2850 2950 50  0001 C CNN
+F 1 "+24V" H 2865 3273 50  0000 C CNN
+F 2 "" H 2850 3100 50  0001 C CNN
+F 3 "" H 2850 3100 50  0001 C CNN
+	1    2850 3100
+	1    0    0    -1
+$EndComp
+$Comp
+L power:+24V #PWR?
+U 1 1 5FAD0834
+P 10350 4600
+AR Path="/5FAD0834" Ref="#PWR?"  Part="1"
+AR Path="/5F71FE73/5FAD0834" Ref="#PWR0108"  Part="1"
+F 0 "#PWR0108" H 10350 4450 50  0001 C CNN
+F 1 "+24V" H 10365 4773 50  0000 C CNN
+F 2 "" H 10350 4600 50  0001 C CNN
+F 3 "" H 10350 4600 50  0001 C CNN
+	1    10350 4600
+	1    0    0    -1
+$EndComp
+$Comp
+L power:+BATT #PWR0109
+U 1 1 5FB47986
+P 7800 850
+F 0 "#PWR0109" H 7800 700 50  0001 C CNN
+F 1 "+BATT" H 7815 1023 50  0000 C CNN
+F 2 "" H 7800 850 50  0001 C CNN
+F 3 "" H 7800 850 50  0001 C CNN
+	1    7800 850
+	1    0    0    -1
+$EndComp
 $EndSCHEMATC

Commit message: New power banana jacks, general updates
Parts:
- removed J1: Conn_01x02_Female, TerminalBlock_Phoenix:TerminalBlock_Phoenix_MKDS-1,5-2-5.08_1x02_P5.08mm_Horizontal, symbol Connector:Conn_01x02_Female
- added C29: 10n, Capacitor_SMD:C_0805_2012Metric, symbol Device:C
- added J1, J6: Conn_01x01_Female, battery-storage-device:banana_jack_right_angle, symbol Connector:Conn_01x01_Female
- added R50: 10M, Resistor_SMD:R_0805_2012Metric, symbol Device:R_US
- added R51: 2M, Resistor_SMD:R_0805_2012Metric, symbol Device:R_US
- added R52: 10k, Resistor_SMD:R_0805_2012Metric, symbol Device:R_US
- added TP6: TestPoint, TestPoint:TestPoint_THTPad_D2.0mm_Drill1.0mm, symbol Connector:TestPoint
- J2: footprint Connector_PinHeader_2.54mm:PinHeader_1x07_P2.54mm_Vertical -> Connector_PinHeader_2.54mm:PinHeader_1x07_P2.54mm_Horizontal
- U7: symbol Analog_ADC:ADS1220xPW -> Battery_Storage_Device-rescue:ADS1220xPW-Analog_ADC
Connections:
- net +5V: now also R52.2
- net +BATT: now also TP6.1
- net ADC_CS: now also R52.1
- net GND: now also C29.2, J6.1 (Pin_1), R51.1; no longer U7.6 (AIN3/REFN1)
- net PACK_HI: now also J1.1 (Pin_1)
- net VC0: now also J2.7 (Pin_7); no longer J2.1 (Pin_1)
- net VC1: now also J2.6 (Pin_6); no longer J2.2 (Pin_2)
- net VC2: now also J2.5 (Pin_5); no longer J2.3 (Pin_3)
- net VC4: now also J2.3 (Pin_3); no longer J2.5 (Pin_5)
- net VC5: now also J2.2 (Pin_2); no longer J2.6 (Pin_6)
- net VC6: now also J2.1 (Pin_1); no longer J2.7 (Pin_7)
- new net: C29.1, R50.1, R51.2, U7.6 (AIN3/REFN1)
- new net RELAY_OUT: R50.2
Other:
- moved on the sheet: C18, C28, R41, R47, R48, U5D, U8

Commit message: Specify exact pin header part number
Parts:
- J2: value Conn_01x07_Male -> TSW-107-08-L-S-RA
Changed lines of the file:
@@
 P 900 1850
 F 0 "J2" H 1008 2331 50  0000 C CNN
-F 1 "Conn_01x07_Male" H 1008 2240 50  0001 C CNN
+F 1 "TSW-107-08-L-S-RA" H 1008 2240 50  0001 C CNN
 F 2 "Connector_PinHeader_2.54mm:PinHeader_1x07_P2.54mm_Horizontal" H 900 1850 50  0001 C CNN
 F 3 "~" H 900 1850 50  0001 C CNN
